Commit message: campero pinza, stop robot con velocidad max, errores arreglados

File: src/description/ur10_campero_pen.urdf.xacro (robot description, xacro)
@@ -15,10 +15,8 @@
 	<!-- Include UR-10 ARM -->
 	<xacro:include filename="$(find ur10_description)/urdf/ur10.urdf.xacro" />
-	<!--xacro:include filename="/home/nacho8/ROS_workspaces/campero_ur10_ws/src/description/ur_description/urdf/ur10.urdf.xacro" /-->
 	<!-- Include force sensor description -->
 	<xacro:include filename="$(find campero_description)/urdf/robotiq_force_torque_sensor/robotiq_fts300.urdf.xacro"/>
 	<!-- Include gripper description -->
     <xacro:include filename="$(find campero_description)/urdf/robotiq_c2/robotiq_85_gripper.urdf.xacro" />
-	<!--xacro:include filename="$(find campero_description)/urdf/robotiq_s/s-model_articulated_macro.xacro"/-->
 	<!-- Wheel parameters -->
 	<xacro:property name="wheel_offset_x" value="0.26" />    <!-- x,y,z in translation from base_link to the center of the wheel -->
@@ -122,18 +120,10 @@
 		  <child link="$(arg prefix)ur10_base_link" />
 		</joint>
-		<!--Lo siguiente comentado es para la pinza-->
-		<!-- UR10 -> robotiq_fts300 -> 2/3f GRIPPER -->
-		<!-- ROBOTIQ SENSOR -->
+		<!--Lo siguiente es para la pinza-->
+		<!-- UR10 -> 2f GRIPPER -->
+        <!-- ROBOTIQ SENSOR -->
 		<xacro:robotiq_fts300 prefix="$(arg prefix)sensor_" parent="$(arg prefix)ur10_ee_link">
-			<origin xyz="0.0 0 0" rpy="0 -1.57 ${pi}"/>
+			<origin xyz="0 0 0" rpy="0 -1.57 ${pi}"/>
 		</xacro:robotiq_fts300>
-		<!-- ROBOTIQ 3f GRIPPER -->
-		<!--xacro:s-model_articulated prefix="$(arg prefix)">
-		</xacro:s-model_articulated-->
-		<!--joint name="$(arg prefix)palm_joint" type="fixed">
-		  <origin xyz="0 0 0.05" rpy="1.57 0 0"/>
-		  <parent link="$(arg prefix)sensor_fts_toolside" />
-		  <child link="$(arg prefix)palm" />
-		</joint-->
 		<!-- ROBOTIQ 85 GRIPPER -->
 		<xacro:robotiq_85_gripper prefix="$(arg prefix)" parent="$(arg prefix)sensor_fts_toolside">
