Commit message: añadido rutas relativas

File: src/description/ur10_campero.urdf.xacro (robot description, xacro)
@@ -14,6 +14,6 @@
 	<xacro:property name="PI" value="3.1415926535897931"/>
 	<!-- Include UR-10 ARM -->
-	<!-- xacro:include filename="$(find ur_description)/urdf/ur10.urdf.xacro" /-->
-	<xacro:include filename="/home/nacho8/ROS_workspaces/campero_ur10_ws/src/description/ur_description/urdf/ur10.urdf.xacro" />
+	<xacro:include filename="$(find ur10_description)/urdf/ur10.urdf.xacro" />
+	<!--xacro:include filename="/home/nacho8/ROS_workspaces/campero_ur10_ws/src/description/ur_description/urdf/ur10.urdf.xacro" /-->
 	<!-- Include force sensor description -->
 	<!--xacro:include filename="$(find campero_description)/urdf/robotiq_force_torque_sensor/robotiq_fts300.urdf.xacro"/-->
@@ -106,5 +106,5 @@
 		</xacro:sensor_axis_m5525>
 		<!-- UR-10 ARM -->
-		<xacro:arg name="kinematics_config" default="$(find ur_description)/config/ur10_default.yaml"/>
+		<xacro:arg name="kinematics_config" default="$(find ur10_description)/config/ur10_default.yaml"/>
 		<xacro:ur10_robot prefix="$(arg prefix)ur10_" joint_limited="true"
 			shoulder_pan_lower_limit="${-PI}" shoulder_pan_upper_limit="${PI}"

File: src/description/ur10_description/urdf/ur10.urdf.xacro (robot description, xacro)
@@ -5,6 +5,6 @@
   Contributers: Jimmy Da Silva, Ajit Krisshna N L, Muhammad Asif Rana
 -->
-  <xacro:include filename="$(find ur_description)/urdf/ur.transmission.xacro" />
-  <xacro:include filename="$(find ur_description)/urdf/ur.gazebo.xacro" />
+  <xacro:include filename="$(find ur10_description)/urdf/ur.transmission.xacro" />
+  <xacro:include filename="$(find ur10_description)/urdf/ur.gazebo.xacro" />
   <xacro:macro name="cylinder_inertial" params="radius length mass *origin">
     <inertial>
@@ -50,5 +50,5 @@
     <xacro:property name="elbow_offset" value="0.049042" /> <!-- measured from model -->
     <xacro:property name="upper_arm_inertia_offset" value="0.175" />  <!-- measured from model -->
-    <!-- This is for compatibility reasons, as transformation between base and base_link was always 180 degree in the ur_description -->
+    <!-- This is for compatibility reasons, as transformation between base and base_link was always 180 degree in the ur10_description -->
     <xacro:property name="base_correction" value="${pi}" />
     <link name="${prefix}base_link" >
@@ -56,5 +56,5 @@
         <origin xyz="0 0 0" rpy="0 0 ${base_correction}"/>
         <geometry>
-          <mesh filename="package://ur_description/meshes/ur10/visual/base.dae"/>
+          <mesh filename="package://ur10_description/meshes/ur10/visual/base.dae"/>
         </geometry>
         <material name="LightGrey">
@@ -65,5 +65,5 @@
         <origin xyz="0 0 0" rpy="0 0 ${base_correction}"/>
         <geometry>
-          <mesh filename="package://ur_description/meshes/ur10/collision/base.stl"/>
+          <mesh filename="package://ur10_description/meshes/ur10/collision/base.stl"/>
         </geometry>
       </collision>
@@ -95,5 +95,5 @@
         <origin xyz="0 0 0" rpy="0 0 ${pi}"/>
         <geometry>
-          <mesh filename="package://ur_description/meshes/ur10/visual/shoulder.dae"/>
+          <mesh filename="package://ur10_description/meshes/ur10/visual/shoulder.dae"/>
         </geometry>
         <material name="LightGrey">
@@ -104,5 +104,5 @@
         <origin xyz="0 0 0" rpy="0 0 ${pi}"/>
         <geometry>
-          <mesh filename="package://ur_description/meshes/ur10/collision/shoulder.stl"/>
+          <mesh filename="package://ur10_description/meshes/ur10/collision/shoulder.stl"/>
         </geometry>
       </collision>
@@ -134,5 +134,5 @@
         <origin xyz="0 0 ${shoulder_offset}" rpy="${pi/2} 0 ${-pi/2}"/>
         <geometry>
-          <mesh filename="package://ur_description/meshes/ur10/visual/upperarm.dae"/>
+          <mesh filename="package://ur10_description/meshes/ur10/visual/upperarm.dae"/>
         </geometry>
         <material name="LightGrey">
@@ -143,5 +143,5 @@
         <origin xyz="0 0 ${shoulder_offset}" rpy="${pi/2} 0 ${-pi/2}"/>
         <geometry>
-          <mesh filename="package://ur_description/meshes/ur10/collision/upperarm.stl"/>
+          <mesh filename="package://ur10_description/meshes/ur10/collision/upperarm.stl"/>
         </geometry>
       </collision>
@@ -173,5 +173,5 @@
         <origin xyz="0 0 ${elbow_offset}" rpy="${pi/2} 0 ${-pi/2}"/>
         <geometry>
-          <mesh filename="package://ur_description/meshes/ur10/visual/forearm.dae"/>
+          <mesh filename="package://ur10_description/meshes/ur10/visual/forearm.dae"/>
         </geometry>
         <material name="LightGrey">
@@ -182,5 +182,5 @@
         <origin xyz="0 0 ${elbow_offset}" rpy="${pi/2} 0 ${-pi/2}"/>
         <geometry>
-          <mesh filename="package://ur_description/meshes/ur10/collision/forearm.stl"/>
+          <mesh filename="package://ur10_description/meshes/ur10/collision/forearm.stl"/>
         </geometry>
       </collision>
@@ -212,5 +212,5 @@
         <origin xyz="0 0 -0.1149" rpy="${pi/2} 0 0"/>
         <geometry>
-          <mesh filename="package://ur_description/meshes/ur10/visual/wrist1.dae"/>
+          <mesh filename="package://ur10_description/meshes/ur10/visual/wrist1.dae"/>
         </geometry>
         <material name="LightGrey">
@@ -221,5 +221,5 @@
         <origin xyz="0 0 -0.1149" rpy="${pi/2} 0 0"/>
         <geometry>
-          <mesh filename="package://ur_description/meshes/ur10/collision/wrist1.stl"/>
+          <mesh filename="package://ur10_description/meshes/ur10/collision/wrist1.stl"/>
         </geometry>
       </collision>
@@ -251,5 +251,5 @@
         <origin xyz="0 0 -0.1158" rpy="0 0 0"/>
         <geometry>
-          <mesh filename="package://ur_description/meshes/ur10/visual/wrist2.dae"/>
+          <mesh filename="package://ur10_description/meshes/ur10/visual/wrist2.dae"/>
         </geometry>
         <material name="LightGrey">
@@ -260,5 +260,5 @@
         <origin xyz="0 0 -0.1158" rpy="0 0 0"/>
         <geometry>
-          <mesh filename="package://ur_description/meshes/ur10/collision/wrist2.stl"/>
+          <mesh filename="package://ur10_description/meshes/ur10/collision/wrist2.stl"/>
         </geometry>
       </collision>
@@ -290,5 +290,5 @@
         <origin xyz="0 0 -0.0922" rpy="${pi/2} 0 0"/>
         <geometry>
-          <mesh filename="package://ur_description/meshes/ur10/visual/wrist3.dae"/>
+          <mesh filename="package://ur10_description/meshes/ur10/visual/wrist3.dae"/>
         </geometry>
         <material name="LightGrey">
@@ -299,5 +299,5 @@
         <origin xyz="0 0 -0.0922" rpy="${pi/2} 0 0"/>
         <geometry>
-          <mesh filename="package://ur_description/meshes/ur10/collision/wrist3.stl"/>
+          <mesh filename="package://ur10_description/meshes/ur10/collision/wrist3.stl"/>
         </geometry>
       </collision>

File: src/description/ur10_description/urdf/ur10_joint_limited_robot.urdf.xacro (robot description, xacro)
@@ -4,9 +4,9 @@
   <xacro:arg name="transmission_hw_interface" default="hardware_interface/PositionJointInterface"/>
   <!-- common stuff -->
-  <xacro:include filename="$(find ur_description)/urdf/common.gazebo.xacro" />
+  <xacro:include filename="$(find ur10_description)/urdf/common.gazebo.xacro" />
   <!-- ur10 -->
-  <xacro:include filename="$(find ur_description)/urdf/ur10.urdf.xacro" />
+  <xacro:include filename="$(find ur10_description)/urdf/ur10.urdf.xacro" />
   <!-- arm -->
-  <xacro:arg name="kinematics_config" default="$(find ur_description)/config/ur10_default.yaml"/>
+  <xacro:arg name="kinematics_config" default="$(find ur10_description)/config/ur10_default.yaml"/>
   <xacro:ur10_robot prefix="" joint_limited="true"
     shoulder_pan_lower_limit="${-pi}" shoulder_pan_upper_limit="${pi}"

File: src/description/ur10_description/urdf/ur10_robot.urdf.xacro (robot description, xacro)
@@ -4,9 +4,9 @@
   <xacro:arg name="transmission_hw_interface" default="hardware_interface/PositionJointInterface"/>
   <!-- common stuff -->
-  <xacro:include filename="$(find ur_description)/urdf/common.gazebo.xacro" />
+  <xacro:include filename="$(find ur10_description)/urdf/common.gazebo.xacro" />
   <!-- ur10 -->
-  <xacro:include filename="$(find ur_description)/urdf/ur10.urdf.xacro" />
+  <xacro:include filename="$(find ur10_description)/urdf/ur10.urdf.xacro" />
   <!-- arm -->
-  <xacro:arg name="kinematics_config" default="$(find ur_description)/config/ur10_default.yaml"/>
+  <xacro:arg name="kinematics_config" default="$(find ur10_description)/config/ur10_default.yaml"/>
   <xacro:ur10_robot prefix="" joint_limited="false"
     transmission_hw_interface="$(arg transmission_hw_interface)"

Commit message: campero_ur10_pen corregido

File: src/description/ur10_campero.urdf.xacro (robot description, xacro)
@@ -15,9 +15,7 @@
 	<!-- Include UR-10 ARM -->
 	<xacro:include filename="$(find ur10_description)/urdf/ur10.urdf.xacro" />
-	<!--xacro:include filename="/home/nacho8/ROS_workspaces/campero_ur10_ws/src/description/ur_description/urdf/ur10.urdf.xacro" /-->
 	<!-- Include force sensor description -->
-	<xacro:include filename="$(find campero_description)/urdf/robotiq_force_torque_sensor/robotiq_fts300.urdf.xacro"/>
+	<!--xacro:include filename="$(find campero_description)/urdf/robotiq_force_torque_sensor/robotiq_fts300.urdf.xacro"/-->
 	<!-- Include gripper description -->
-    <xacro:include filename="$(find campero_description)/urdf/robotiq_c2/robotiq_85_gripper.urdf.xacro" />
 	<!--xacro:include filename="$(find campero_description)/urdf/robotiq_s/s-model_articulated_macro.xacro"/-->
 	<!-- Wheel parameters -->
@@ -125,7 +123,7 @@
 		<!-- UR10 -> robotiq_fts300 -> 2/3f GRIPPER -->
 		<!-- ROBOTIQ SENSOR -->
-		<xacro:robotiq_fts300 prefix="$(arg prefix)sensor_" parent="$(arg prefix)ur10_ee_link">
+		<!--xacro:robotiq_fts300 prefix="$(arg prefix)sensor_" parent="$(arg prefix)ur10_ee_link">
 			<origin xyz="0.0 0 0" rpy="0 -1.57 ${pi}"/>
-		</xacro:robotiq_fts300>
+		</xacro:robotiq_fts300-->
 		<!-- ROBOTIQ 3f GRIPPER -->
 		<!--xacro:s-model_articulated prefix="$(arg prefix)">
@@ -136,8 +134,4 @@
 		  <child link="$(arg prefix)palm" />
 		</joint-->
-		<!-- ROBOTIQ 85 GRIPPER -->
-		<xacro:robotiq_85_gripper prefix="$(arg prefix)" parent="$(arg prefix)sensor_fts_toolside">
-			<origin xyz="0 0.0 0" rpy="0 -1.57 0"/>
-		</xacro:robotiq_85_gripper>
    </xacro:macro>
    <xacro:ros_control/>
