Commit message: permite pizarras distinto tamaño

File: src/campero_ur10/description/campero_ur10_description/robots/campero_ur10.urdf.xacro (robot description, xacro)
@@ -164,5 +164,5 @@
 			<visual> <!-- cylinder -->
 				<!--xyz = "? box2.size.y/2-box1.size.y/2 box1.size.y/2 - box2.size.z/2"-->
-				<origin xyz=" 0.04 0.02 0.045" rpy="0 ${PI*1/2} 0" />
+				<origin xyz=" 0.04 0.03 0.045" rpy="0 ${PI*1/2} 0" />
 				<geometry>
 					<cylinder length="0.24" radius="0.01"/>

Commit message: init aruco, realsense

File: src/campero_ur10/description/campero_ur10_description/robots/campero_ur10.urdf.xacro (robot description, xacro)
@@ -134,5 +134,5 @@
 		<!-- Real sense camara D435 -->
 		<xacro:sensor_d435 parent="ee_link">
-			<origin xyz="0.05 0 -0.04" rpy="${PI} 0 0"/>
+			<origin xyz="0.055 0 -0.045" rpy="${PI} 0 0"/>
 		</xacro:sensor_d435>
 		<!-- Soporte rotulador -->
@@ -140,5 +140,5 @@
 			<parent link ="ee_link" />
 			<child link = "base_pen_link" />
-			<origin xyz="0.08 0.0 0.1" rpy="0.0 0.0 0.0" />
+			<origin xyz="0.08 0.0 0.09" rpy="0.0 0.0 0.0" />
 		</joint>
 		<link name = "base_pen_link" type="fixed">
@@ -146,5 +146,5 @@
 				<origin xyz=" 0 0 0" rpy="0 0 0" />
 				<geometry>
-					<box size="0.01 0.04 0.13"/>
+					<box size="0.01 0.045 0.115"/>
 				</geometry>
 				<material name="grey">
@@ -153,8 +153,8 @@
 			</visual>
 			<visual> <!-- box2 -->
-				<!--xyz = "box2.size.x/2-box1.size.x/2 box2.size.y/2-box1.size.y/2 box1.size.y/2 - box2.size.z/2"-->
-				<origin xyz=" 0.015 0.02 0.045" rpy="0 0 0" />
+				<!--xyz = "box2.size.x/2-box1.size.x/2 box2.size.y/2+box1.size.y/2 box1.size.z/2 - box2.size.z/2"-->
+				<origin xyz=" 0.011 0.0475 0.0375" rpy="0 0 0" />
 				<geometry>
-					<box size="0.04 0.08 0.04"/>
+					<box size="0.032 0.05 0.04"/>
 				</geometry>
 				<material name="black">
@@ -164,7 +164,7 @@
 			<visual> <!-- cylinder -->
 				<!--xyz = "? box2.size.y/2-box1.size.y/2 box1.size.y/2 - box2.size.z/2"-->
-				<origin xyz=" 0.04 0.03 0.045" rpy="0 ${PI*1/2} 0" />
+				<origin xyz=" 0.04 0.0475 0.0375" rpy="0 ${PI*1/2} 0" />
 				<geometry>
-					<cylinder length="0.24" radius="0.01"/>
+					<cylinder length="0.25" radius="0.0075"/>
 				</geometry>
 				<material name="yellow">

Commit message: calib sim ok, pts img -> world ok

File: src/campero_ur10/description/campero_ur10_description/robots/campero_ur10.urdf.xacro (robot description, xacro)
@@ -137,38 +137,77 @@
 		</xacro:sensor_d435>
 		<!-- Soporte rotulador -->
-		<joint name="base_pen_joint" type="fixed">
+		<!--joint name="base_pen_joint" type="fixed">
 			<parent link ="ee_link" />
 			<child link = "base_pen_link" />
-			<origin xyz="0.08 0.0 0.09" rpy="0.0 0.0 0.0" />
+			<origin xyz="0.286 0.04 0.113 " rpy="0.0 0.0 0.0" />
 		</joint>
 		<link name = "base_pen_link" type="fixed">
-			<visual> <!-- box1 -->
-				<origin xyz=" 0 0 0" rpy="0 0 0" />
-				<geometry>
-					<box size="0.01 0.045 0.115"/>
-				</geometry>
-				<material name="grey">
-					<color rgba="0.5 0.5 0.5 1"/>
-				</material>
-			</visual>
-			<visual> <!-- box2 -->
-				<!--xyz = "box2.size.x/2-box1.size.x/2 box2.size.y/2+box1.size.y/2 box1.size.z/2 - box2.size.z/2"-->
-				<origin xyz=" 0.011 0.0475 0.0375" rpy="0 0 0" />
-				<geometry>
-					<box size="0.032 0.05 0.04"/>
-				</geometry>
-				<material name="black">
-					<color rgba="0 0 0 1"/>
-				</material>
-			</visual>
-			<visual> <!-- cylinder -->
-				<!--xyz = "? box2.size.y/2-box1.size.y/2 box1.size.y/2 - box2.size.z/2"-->
-				<origin xyz=" 0.04 0.0475 0.0375" rpy="0 ${PI*1/2} 0" />
-				<geometry>
-					<cylinder length="0.25" radius="0.0075"/>
+			<visual> <!- cilindro soporte ->
+				<!-xyz = "0 0 -lenght/2"->
+				<origin xyz="-0.14 0 0" rpy="0 ${PI/2} 0" />
+				<geometry>
+					<cylinder length="0.24" radius="0.0075"/>
 				</geometry>
 				<material name="yellow">
                 	<color rgba="1 0.4 0 1"/>
             	</material>
+			</visual>
+			<visual> <!- box ->
+				<!-xyz = "-0 0 -(cilindro.lenght-0.04-size.z/2)"->
+				<origin xyz="-0.205 0 0" rpy="0 0 0" />
+				<geometry>
+					<box size="0.04 0.04 0.04 "/>
+				</geometry>
+				<material name="black">
+					<color rgba="0 0 0 1"/>
+				</material>
+			</visual>
+			<visual> <!-conector wrist3->
+				<!-xyz = "-offset_ee_punta.x box.size.y/2 medida"->
+				<origin xyz="-0.22 -0.04 -0.02" rpy="0 0 0" />
+				<geometry>
+					<box size="0.01 0.045 0.08"/>
+				</geometry>
+				<material name="grey">
+					<color rgba="0.5 0.5 0.5 1"/>
+				</material>
+			</visual>
+  		</link-->
+		<!-- Soporte rotulador -->
+		<joint name="base_pen_joint" type="fixed">
+			<parent link ="wrist_3_link" />
+			<child link = "base_pen_link" />
+			<origin xyz="-0.04 -0.113 0.286" rpy="0.0 0.0 0.0" />
+		</joint>
+		<link name = "base_pen_link" type="fixed">
+			<visual> <!--cilindro soporte-->
+				<!--xyz = "0 0 -lenght/2"-->
+				<origin xyz="0 0 -0.14" rpy="0 0 0" />
+				<geometry>
+					<cylinder length="0.24" radius="0.0075"/>
+				</geometry>
+				<material name="yellow">
+                	<color rgba="1 0.4 0 1"/>
+            	</material>
+			</visual>
+			<visual> <!--box-->
+				<!--xyz = "-0 0 -(cilindro.lenght-0.04-size.z/2)"-->
+				<origin xyz="0 0 -0.205" rpy="0 0 0" />
+				<geometry>
+					<box size="0.04 0.04 0.04 "/>
+				</geometry>
+				<material name="black">
+					<color rgba="0 0 0 1"/>
+				</material>
+			</visual>
+			<visual> <!--conector wrist3-->
+				<!--xyz = "-offset_ee_punta.x box.size.y/2 medida"-->
+				<origin xyz="0.04 0.02 -0.22" rpy="0 0 0" />
+				<geometry>
+					<box size="0.045 0.08 0.01"/>
+				</geometry>
+				<material name="grey">
+					<color rgba="0.5 0.5 0.5 1"/>
+				</material>
 			</visual>
   		</link>

Commit message: draw img ok

File: src/campero_ur10/description/campero_ur10_description/robots/campero_ur10.urdf.xacro (robot description, xacro)
@@ -178,10 +178,10 @@
 			<parent link ="wrist_3_link" />
 			<child link = "base_pen_link" />
-			<origin xyz="-0.04 -0.113 0.286" rpy="0.0 0.0 0.0" />
+			<origin xyz="-0.04 -0.13 0.26" rpy="0.0 0.0 0.0" />
 		</joint>
 		<link name = "base_pen_link" type="fixed">
 			<visual> <!--cilindro soporte-->
 				<!--xyz = "0 0 -lenght/2"-->
-				<origin xyz="0 0 -0.14" rpy="0 0 0" />
+				<origin xyz="0 0 -0.11" rpy="0 0 0" />
 				<geometry>
 					<cylinder length="0.24" radius="0.0075"/>
@@ -193,5 +193,5 @@
 			<visual> <!--box-->
 				<!--xyz = "-0 0 -(cilindro.lenght-0.04-size.z/2)"-->
-				<origin xyz="0 0 -0.205" rpy="0 0 0" />
+				<origin xyz="0 0 -0.175" rpy="0 0 0" />
 				<geometry>
 					<box size="0.04 0.04 0.04 "/>
@@ -203,5 +203,5 @@
 			<visual> <!--conector wrist3-->
 				<!--xyz = "-offset_ee_punta.x box.size.y/2 medida"-->
-				<origin xyz="0.04 0.02 -0.22" rpy="0 0 0" />
+				<origin xyz="0.04 0.02 -0.19" rpy="0 0 0" />
 				<geometry>
 					<box size="0.045 0.08 0.01"/>

Commit message: limpieza 1

File: src/campero_ur10/description/campero_ur10_description/robots/campero_ur10.urdf.xacro (robot description, xacro)
@@ -136,52 +136,13 @@
 			<origin xyz="0.055 0 -0.045" rpy="${PI} 0 0"/>
 		</xacro:sensor_d435>
-		<!-- Soporte rotulador -->
-		<!--joint name="base_pen_joint" type="fixed">
+		<!--Soporte rotulador-->
+		<joint name="base_pen_joint" type="fixed">
 			<parent link ="ee_link" />
 			<child link = "base_pen_link" />
-			<origin xyz="0.286 0.04 0.113 " rpy="0.0 0.0 0.0" />
-		</joint>
-		<link name = "base_pen_link" type="fixed">
-			<visual> <!- cilindro soporte ->
-				<!-xyz = "0 0 -lenght/2"->
-				<origin xyz="-0.14 0 0" rpy="0 ${PI/2} 0" />
-				<geometry>
-					<cylinder length="0.24" radius="0.0075"/>
-				</geometry>
-				<material name="yellow">
-                	<color rgba="1 0.4 0 1"/>
-            	</material>
-			</visual>
-			<visual> <!- box ->
-				<!-xyz = "-0 0 -(cilindro.lenght-0.04-size.z/2)"->
-				<origin xyz="-0.205 0 0" rpy="0 0 0" />
-				<geometry>
-					<box size="0.04 0.04 0.04 "/>
-				</geometry>
-				<material name="black">
-					<color rgba="0 0 0 1"/>
-				</material>
-			</visual>
-			<visual> <!-conector wrist3->
-				<!-xyz = "-offset_ee_punta.x box.size.y/2 medida"->
-				<origin xyz="-0.22 -0.04 -0.02" rpy="0 0 0" />
-				<geometry>
-					<box size="0.01 0.045 0.08"/>
-				</geometry>
-				<material name="grey">
-					<color rgba="0.5 0.5 0.5 1"/>
-				</material>
-			</visual>
-  		</link-->
-		<!-- Soporte rotulador -->
-		<joint name="base_pen_joint" type="fixed">
-			<parent link ="wrist_3_link" />
-			<child link = "base_pen_link" />
-			<origin xyz="-0.04 -0.13 0.26" rpy="0.0 0.0 0.0" />
+			<origin xyz="0.264 0.0435 0.129" rpy="0.0 0.0 0.0" />
 		</joint>
 		<link name = "base_pen_link" type="fixed">
 			<visual> <!--cilindro soporte-->
-				<!--xyz = "0 0 -lenght/2"-->
-				<origin xyz="0 0 -0.11" rpy="0 0 0" />
+				<origin xyz="-0.11 0 0" rpy="0 ${PI/2} 0" />
 				<geometry>
 					<cylinder length="0.24" radius="0.0075"/>
@@ -192,6 +153,5 @@
 			</visual>
 			<visual> <!--box-->
-				<!--xyz = "-0 0 -(cilindro.lenght-0.04-size.z/2)"-->
-				<origin xyz="0 0 -0.175" rpy="0 0 0" />
+				<origin xyz="-0.175 0 0" rpy="0 0 0" />
 				<geometry>
 					<box size="0.04 0.04 0.04 "/>
@@ -202,8 +162,7 @@
 			</visual>
 			<visual> <!--conector wrist3-->
-				<!--xyz = "-offset_ee_punta.x box.size.y/2 medida"-->
-				<origin xyz="0.04 0.02 -0.19" rpy="0 0 0" />
+				<origin xyz="-0.19 -0.04 -0.035" rpy="0 0 0" />
 				<geometry>
-					<box size="0.045 0.08 0.01"/>
+					<box size="0.01 0.045 0.11"/>
 				</geometry>
 				<material name="grey">

Commit message: limpieza 2

File: src/campero_ur10/description/campero_ur10_description/robots/campero_ur10.urdf.xacro (robot description, xacro)
@@ -144,5 +144,5 @@
 		<link name = "base_pen_link" type="fixed">
 			<visual> <!--cilindro soporte-->
-				<origin xyz="-0.11 0 0" rpy="0 ${PI/2} 0" />
+				<origin xyz="-0.13 0 0" rpy="0 ${PI/2} 0" />
 				<geometry>
 					<cylinder length="0.24" radius="0.0075"/>
